File: servolicious.kicad_pcb (KiCad board)
At the start: 2 copper layers, 57.5 x 27.5 mm, 14 parts, among them J1 Conn_01x03_Pin, J10 Barrel_Jack_MountingPin, J2 Conn_01x03_Pin, J3 Conn_01x03_Pin, J4 Conn_01x03_Pin, J5 Conn_01x03_Pin, J6 Conn_01x03_Pin, J7 Conn_01x03_Pin, J8 Conn_01x03_Pin, J9 Conn_01x03_Pin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

Commit message: Servo headers were wrong
Connections:
- J1 pad 1: +5V -> Earth
- J1 pad 2: /Servo1 -> +5V
- J1 pad 3: Earth -> /Servo1
- J2 pad 1: +5V -> Earth
- J2 pad 2: /Servo2 -> +5V
- J2 pad 3: Earth -> /Servo2
- J3 pad 1: +5V -> Earth
- J3 pad 2: /Servo3 -> +5V
- J3 pad 3: Earth -> /Servo3
- J4 pad 1: +5V -> Earth
- J4 pad 2: /Servo4 -> +5V
- J4 pad 3: Earth -> /Servo4
- J5 pad 1: +5V -> Earth
- J5 pad 2: /Servo5 -> +5V
- J5 pad 3: Earth -> /Servo5
- J6 pad 1: +5V -> Earth
- J6 pad 2: /Servo6 -> +5V
- J6 pad 3: Earth -> /Servo6
- J7 pad 1: +5V -> Earth
- J7 pad 2: /Servo7 -> +5V
- J7 pad 3: Earth -> /Servo7
- J8 pad 1: +5V -> Earth
- J8 pad 2: /Servo8 -> +5V
- J8 pad 3: Earth -> /Servo8
Routing:
- net /Servo5: track 10.5 -> 7.95 mm
- net /Servo4: track 17.0 -> 14.5 mm
- net /Servo8: track 25.7 -> 27.6 mm
- net /Servo1: track 24.8 -> 23.7 mm
- net /Servo2: track 21.3 -> 20.3 mm
- net /Servo3: track 18.6 -> 17.5 mm
- net /Servo6: track 14.8 -> 15.5 mm
