File: servolicious.kicad_sch (KiCad schematic)
At the start: 29 parts, among them J1 Conn_01x03_Pin, J10 Conn_01x03_Pin, J11 Conn_01x03_Pin, J12 Conn_01x03_Pin, J13 Conn_01x03_Pin, J14 Conn_01x03_Pin, J15 Conn_01x03_Pin, J16 Conn_01x03_Pin, J17 Barrel_Jack_MountingPin, J18 Conn_01x03, J2 Conn_01x03_Pin, J3 Conn_01x03_Pin, J4 Conn_01x03_Pin, J5 Conn_01x03_Pin, J6 Conn_01x03_Pin, J7 Conn_01x03_Pin, J8 Conn_01x03_Pin, J9 Conn_01x03_Pin, U2 PCA9685PW

Commit message: Interactive PWM control for finer grained management of servos
Parts:
- removed J18: Conn_01x03, Connector_PinSocket_2.54mm:PinSocket_1x03_P2.54mm_Vertical, symbol Connector_Generic:Conn_01x03
- added J18: Conn_01x05, Connector_PinHeader_2.54mm:PinHeader_1x05_P2.54mm_Vertical, symbol Connector_Generic:Conn_01x05
- added R1, R2: R_Small, Resistor_SMD:R_0603_1608Metric_Pad0.98x0.95mm_HandSolder, symbol Device:R_Small
Connections:
- net Earth: now also J18.1 (Pin_1), R1.2, R2.2; no longer U2.23 (~{OE})
- net SCL: now also J18.3 (Pin_3)
- net SDA: now also J18.4 (Pin_4)
- net CLK: now reaches U2.25 (EXTCLK)
- net CLK: now also J18.2 (Pin_2), R1.1
- new net OE: J18.5 (Pin_5), R2.1, U2.23 (~{OE})
- no-connect marks 2 -> 1
